File: BandPCB/BigSphereBand.sch (KiCad schematic (older format))
At the start: 102 parts

Commit message: Proceeding
Parts:
- added XL10, XL11, XL12, XL3, XL4, XL5, XL6, XL7, XL8, XL9: CONN_1, PCB:Oval3x1.5, symbol Connectors_kl:CONN_1
- gave numbers to parts that had none: 93
- renumbered C28 to C26, C44 to C36, C52 to C41, C57 to C46, DA4 to DA6, L1 to L6, R20 to R11, R23 to R16
Connections:
- net LED10_CTRL: now also XL12.1 (P1)
- net LED1_CTRL: now also XL3.1 (P1)
- net LED2_CTRL: now also XL4.1 (P1)
- net LED3_CTRL: now also XL5.1 (P1)
- net LED4_CTRL: now also XL6.1 (P1)
- net LED5_CTRL: now also XL7.1 (P1)
- net LED6_CTRL: now also XL8.1 (P1)
- net LED7_CTRL: now also XL9.1 (P1)
- net LED8_CTRL: now also XL10.1 (P1)
- net LED9_CTRL: now also XL11.1 (P1)
