File: BSMainPCB/BSMainPCB.kicad_pcb (KiCad board)
At the start: 2 copper layers, 200 x 126 mm, 1004 parts, among them Q1 2N7002, Q10 IRF9321, Q11 2N7002, Q12 IRF9321, Q13 2N7002, Q14 IRF9321, Q15 2N7002, Q16 IRF9321, Q17 2N7002, Q18 IRF9321, Q2 IRF9321, Q3 2N7002, Q4 IRF9321, Q5 2N7002, Q6 IRF9321, Q7 2N7002, Q8 IRF9321, Q9 2N7002, SW1 SWITCH_H, U1 USBLC6

Commit message: - Lot of capacitors near LEDs removed, as eDesignSuite shows they are not required
Parts:
- removed C100, C101, C102, C103, C104, C105, C106, C107, C108, C109, C110, C111, C170, C171, C172, C173, C174, C175, C176, C177, C178, C179, C180, C181, C182, C183, C242, C243, C244, C245, C246, C247, C248, C249, C250, C251, C252, C253, C254, C255, C314, C315, C316, C317, C318, C319, C320, C321, C322, C323, C324, C325, C326, C327, C357, C358, C359, C360, C361, C362, C363, C98, C99: 0.1u, Capacitors:CAP_0603
- removed C156, C157, C158, C159, C160, C161, C162, C163, C164, C165, C166, C167, C168, C169, C228, C229, C230, C231, C232, C233, C234, C235, C236, C237, C238, C239, C240, C241, C300, C301, C302, C303, C304, C305, C306, C307, C308, C309, C310, C311, C312, C313, C350, C351, C352, C353, C354, C355, C356, C84, C85, C86, C87, C88, C89, C90, C91, C92, C93, C94, C95, C96, C97: 10u, Capacitors:CAP_0805
- moved R18 443.0 mm to (32.0, 44.6), turned to 180 degrees
- moved C71 428.5 mm to (36.0, 143.6), turned to 180 degrees
- moved R229 408.4 mm to (32.0, 46.8), turned to 180 degrees
- moved R228 408.2 mm to (35.0, 46.8), turned to 180 degrees
- moved R19 399.3 mm to (32.0, 38.4), turned to -90 degrees
- moved Q1 367.6 mm to (32.0, 41.8), turned to 180 degrees
- moved XL30 355.5 mm to (91.9, 147.8), turned to -90 degrees
- moved TP45 346.8 mm to (134.2, 47.4)
- moved TP44 342.0 mm to (132.6, 47.4)
- moved Q2 338.3 mm to (36.6, 40.5), turned to 180 degrees
- moved XL41 327.5 mm to (102.6, 147.8), turned to -90 degrees
- moved XL28 327.2 mm to (81.8, 147.8), turned to -90 degrees
- moved TP52 325.8 mm to (145.6, 47.4)
- moved TP47 325.3 mm to (137.4, 47.4)
- moved TP48 325.2 mm to (139.2, 47.4)
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
Commit message: * Hole connection changed
Parts:
- R236, R237, R238, R239, R240, R241, R242, R243, R244, R245, R246, R247, R248, R249, R250, R251, R38, R39, R43, R44, R45, R46, R52, R53, R58, R59, R60, R61, R67, R68: moved to B.Cu
- moved L8 411.8 mm to (40.5, 141.0), turned to 180 degrees
- moved C75 396.0 mm to (51.5, 143.6), turned to 180 degrees
- moved C73 395.3 mm to (40.4, 143.6), turned to 180 degrees
- moved L7 392.2 mm to (34.9, 141.0), turned to 180 degrees
- moved C44 379.2 mm to (39.4, 128.4)
- moved C56 377.3 mm to (28.8, 138.6), turned to 180 degrees
- moved L9 376.7 mm to (46.0, 141.0), turned to 180 degrees
- moved L6 361.1 mm to (29.2, 141.0), turned to 180 degrees
- moved C43 360.1 mm to (33.6, 128.4)
- moved C46 356.8 mm to (50.6, 128.4)
- moved R61 353.4 mm to (45.4, 143.4)
- moved R52 351.4 mm to (51.0, 141.0)
- moved C74 349.9 mm to (46.0, 143.6), turned to 180 degrees
- moved L11 347.5 mm to (57.2, 141.0), turned to 180 degrees
- moved R45 340.3 mm to (39.8, 143.4)
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Connections:
- HOLE10 pad H: GND -> GNDPWR
- HOLE11 pad H: GND -> GNDPWR
- HOLE12 pad H: GND -> GNDPWR
- HOLE9 pad H: GND -> GNDPWR

Commit message: Proceeding with layout
Parts:
- removed HOLE10, HOLE11, HOLE12, HOLE5, HOLE6, HOLE7, HOLE8, HOLE9: HOLE_METALLED, PCB:Hole3_5_out6mm
- added L68: BLM15AG102, Inductors:IND_0402, F.Cu at (54.2, 88.3)
- added Q19: 2N7002, SOT:SOT23-3, F.Cu at (58.0, 52.8)
- added Q20: IRLML9303, SOT:SOT23-3, F.Cu at (61.8, 50.8)
- added R262: 100k, Resistors:RES_0603, F.Cu at (58.0, 50.0)
- added R263: 1k, Resistors:RES_0603, F.Cu at (61.8, 53.6)
- added TP31: TESTPOINT, PCB:TESTPOINT_1MM, F.Cu at (55.4, 52.8)
- added XL79: CONN_2, Connectors:W02_Pitch_2d54, F.Cu at (60.4, 46.2)
- ANT1: footprint Antennas:ANT_868_IFA_SIMPLEJOY -> Antennas:ANT_868_IFA_SIMPLEJOY_MIRR
- C1, C10, C11, C12, C127, C128, C129, C13, C130, C131, C132, C133, C134, C135, C136, C137, C138, C139, C14, C140, C15, C16, C17, C18, C19, C199, C20, C200, C201, C202, C203, C204, C205, C206, C207, C208, C209, C210, C211, C212, C22, C24, C25, C26, C27, C271, C272, C273, C274, C275, C276, C277, C278, C279, C28, C280, C281, C282, C283, C284, C3, C31, C32, C336, C337, C338, C339, C34, C340, C341, C342, C36, C37, C38, C39, C4, C55, C56, C57, C58, C59, C60, C61, C62, C63, C64, C65, C66, C67, C68, C7, C8, C9: footprint Capacitors:CAP_0603 -> Capacitors:CAP_0603_Silks
- C2, C30: value 100u -> 10u; footprint Capacitors:SMD_D6d3 -> Capacitors:CAP_0805
- C21: value 0.1u -> 1u; footprint Capacitors:CAP_0603 -> Capacitors:CAP_0603_Silks
- R102, R103, R106, R107, R108, R109, R110, R116, R117, R87, R88, R91, R92, R93, R94, R95: moved to B.Cu
- moved C37 410.9 mm to (38.3, 58.6)
- moved C25 396.5 mm to (44.8, 87.0), turned to 180 degrees
- moved VCap2 394.9 mm to (46.8, 69.8), turned to 90 degrees
- moved C12 394.7 mm to (45.2, 69.8), turned to 90 degrees
- moved C16 394.1 mm to (41.2, 82.3), turned to 90 degrees
- moved C38 391.8 mm to (43.5, 62.7)
- moved C4 390.9 mm to (41.2, 56.2), turned to -90 degrees
- moved R14 389.7 mm to (49.6, 86.9)
- moved C34 389.6 mm to (33.3, 65.3), turned to 180 degrees
- moved R2 389.6 mm to (28.3, 50.6)
- moved R15 388.9 mm to (43.2, 51.6), turned to 90 degrees
- moved C11 382.0 mm to (35.4, 56.2), turned to 90 degrees
- moved C36 377.9 mm to (33.3, 59.8), turned to 180 degrees
- moved L21 372.9 mm to (74.6, 141.0), turned to 180 degrees
- moved R20 371.8 mm to (50.2, 58.8)
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Connections:
- C2 pad 1: PwrUnst -> GND
- C2 pad 2: GNDPWR -> +3v3
- C20 pad 2: GND -> GNDPWR
- C21 pad 1: PwrMCU -> Net-(C21-Pad1)
- C23 pad 2: GND -> GNDPWR
- C30 pad 1: +3v3 -> PwrUnst
- C30 pad 2: GND -> GNDPWR
- D10 pad C: GND -> GNDPWR
- D11 pad C: GND -> GNDPWR
- D3 pad C: GND -> GNDPWR
- D4 pad C: GND -> GNDPWR
- D5 pad C: GND -> GNDPWR
- D6 pad C: GND -> GNDPWR
- D7 pad C: GND -> GNDPWR
- D8 pad C: GND -> GNDPWR
- D9 pad C: GND -> GNDPWR
- DD2 pad 13: PwrMCU -> Net-(C21-Pad1)
- DD2 pad 2: /LED_PWR8 -> /PWR_CTRL9
- DD2 pad 3: /LED_PWR9 -> /LED_PWR8
- DD2 pad 39: /PWR_CTRL5 -> /VENT_CTRL
- DD2 pad 4: (no net) -> /LED_PWR9
- DD2 pad 40: /PWR_CTRL6 -> /PWR_CTRL5
- DD2 pad 51: /PWR_CTRL7 -> /PWR_CTRL6
- DD2 pad 52: /PWR_CTRL8 -> /PWR_CTRL7
- DD2 pad 53: /PWR_CTRL9 -> /PWR_CTRL8
- HOLE1 pad H: GND -> GNDPWR
- HOLE2 pad H: GND -> GNDPWR
- HOLE3 pad H: GND -> GNDPWR
Other:
- board size 200 x 126 mm -> 200 x 108 mm

Commit message: Proceeding with layout
Parts:
- C112, C141, C184, C213, C23, C256, C285, C335, C40, C69: footprint Capacitors:CAP_10xxR -> Capacitors:CAP_10Rx16_HOR; moved to B.Cu
- R100, R104, R105, R111, R112, R113, R114, R115, R118, R119, R89, R90, R96, R97, R98, R99: moved to B.Cu
- moved C137 340.6 mm to (120.2, 138.6), turned to 180 degrees
- moved L30 333.3 mm to (125.6, 141.0), turned to 180 degrees
- moved C150 325.6 mm to (109.4, 143.6), turned to 180 degrees
- moved C153 318.1 mm to (126.2, 143.6), turned to 180 degrees
- moved L31 313.7 mm to (131.2, 141.0), turned to 180 degrees
- moved C139 309.7 mm to (131.4, 138.6), turned to 180 degrees
- moved L27 305.0 mm to (108.8, 141.0), turned to 180 degrees
- moved L26 301.2 mm to (103.2, 141.0), turned to 180 degrees
- moved C136 281.9 mm to (114.6, 138.6), turned to 180 degrees
- moved C152 270.1 mm to (120.6, 143.6), turned to 180 degrees
- moved R115 269.3 mm to (125.6, 141.0)
- moved R119 267.7 mm to (136.8, 138.6)
- moved L28 263.8 mm to (114.4, 141.0), turned to 180 degrees
- moved L29 254.1 mm to (120.0, 141.0), turned to 180 degrees
- moved C135 252.6 mm to (109.0, 138.6), turned to 180 degrees
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Connections:
- XL4 pad H2: (no net) -> Net-(C1-Pad2)
- XL4 pad H3: (no net) -> Net-(C1-Pad2)
- XL4 pad H4: (no net) -> Net-(C1-Pad2)
Other:
- outline, holes or cut-outs redrawn

Commit message: Layout done
Parts:
- R137, R138, R139, R140, R141, R142, R143, R144, R145, R146, R147, R148, R149, R150, R151, R152, R153, R154, R155, R156, R157, R158, R159, R160, R161, R162, R163, R164, R165, R166, R167, R168, R187, R188, R189, R190, R191, R192, R193, R194, R195, R196, R197, R198, R199, R200, R201, R202, R203, R204, R205, R206, R207, R208, R209, R210, R211, R212, R213, R214, R215, R216, R217, R218, R40, R41, R48, R49, R50, R51, R54, R55, R62, R63, R64, R65, R66, R69, R70: moved to B.Cu
- moved L38 380.9 mm to (71.0, 113.2), turned to 180 degrees
- moved R12 379.2 mm to (43.7, 60.5), turned to 90 degrees
- moved C202 365.4 mm to (60.0, 110.8), turned to 180 degrees
- moved L34 362.1 mm to (48.6, 113.2), turned to 180 degrees
- moved L47 360.5 mm to (83.2, 113.2), turned to 180 degrees
- moved L33 359.1 mm to (43.0, 113.2), turned to 180 degrees
- moved TP11 357.8 mm to (56.2, 76.2)
- moved TP5 353.3 mm to (77.0, 78.2)
- moved R155 352.8 mm to (43.0, 113.2)
- moved TP3 351.4 mm to (42.0, 62.4)
- moved L39 348.1 mm to (76.6, 113.2), turned to 180 degrees
- moved TP1 344.0 mm to (78.4, 64.2)
- moved C275 341.2 mm to (105.8, 110.8), turned to 180 degrees
- moved TP2 337.9 mm to (55.4, 66.0)
- moved C218 337.7 mm to (66.0, 115.8), turned to 180 degrees
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Other:
- board size 200 x 108 mm -> 200 x 99 mm
- copper layers 2 -> 4
